File: Mergung.kicad_pcb (KiCad board)
At the start: 2 copper layers, 41 parts, among them Con1B1 Battery In, M1 80V 77A, M2 80V 77A, M3 80V 77A, M4 100V 200A

Commit message: new component placement, pending review
Parts:
- added Con2: 12V Out, Connector_Wire:SolderWirePad_1x01_SMD_5x10mm, F.Cu at (97.5, 92.5)
- added Con3: 19.5V Out, Connector_Wire:SolderWirePad_1x01_SMD_5x10mm, F.Cu at (97.5, 138.0)
- added U1: LM5149RGYR, LM5149:VQFN24_RGY_TEX, F.Cu at (38.5, 79.8)
- added U2: LM5149RGYR, LM5149:VQFN24_RGY_TEX, F.Cu at (35.2, 131.8)
- moved Rpg2 136.3 mm to (28.8, 137.5)
- moved Rconfig2 127.7 mm to (37.7, 121.5)
- moved Ccomp4 124.3 mm to (31.3, 126.5)
- moved Ccomp3 121.4 mm to (30.3, 122.0)
- moved Rfbb1 116.7 mm to (37.8, 144.0)
- moved Cvcc2 115.9 mm to (31.0, 142.5)
- moved Cboot1 114.9 mm to (39.5, 93.5)
- moved NT1 109.5 mm to (97.0, 111.5), turned to -90 degrees
- moved Rcomp2 108.4 mm to (34.3, 137.9)
- moved Rfbt1 105.4 mm to (42.1, 142.5)
- moved Rvdda1 103.0 mm to (39.5, 98.0)
- moved Rt2 100.3 mm to (37.5, 119.0)
- moved Rt1 92.1 mm to (40.5, 75.0)
- moved Rconfig1 91.5 mm to (40.0, 72.0), turned to 180 degrees
- moved Cvdda2 85.9 mm to (39.5, 147.5)
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Other:
- board text added: "80V -> 12V"
- board text added: "80V -> 19V"
