File: Mergung.kicad_sch (KiCad schematic)
At the start: 45 parts, among them Con1B1 Battery In, Con2 12V Out, Con3 19.5V Out, M1 80V 77A, M2 80V 77A, M3 80V 77A, M4 100V 200A, U1 LM5149RGYR, U2 LM5149RGYR

Commit message: added 1 footprint
Parts:
- NT1: footprint (none) -> NetTie:NetTie-2_SMD_Pad2.0mm
Changed lines of the file:
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@@
 			)
 		)
-		(property "Footprint" ""
+		(property "Footprint" "NetTie:NetTie-2_SMD_Pad2.0mm"
 			(at 33.02 92.71 0)
 			(effects

Commit message: new component placement, pending review
Parts:
- Con1B1: footprint (none) -> Connector_Wire:SolderWirePad_1x01_SMD_5x10mm
- Con2, Con3: footprint Wire Holes:Vout Holed -> Connector_Wire:SolderWirePad_1x01_SMD_5x10mm
Changed lines of the file:
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@@
 			)
 		)
-		(property "Footprint" "Wire Holes:Vout Holed"
+		(property "Footprint" "Connector_Wire:SolderWirePad_1x01_SMD_5x10mm"
 			(at 257.81 156.21 0)
 			(effects
@@
 			)
 		)
-		(property "Footprint" ""
+		(property "Footprint" "Connector_Wire:SolderWirePad_1x01_SMD_5x10mm"
 			(at 43.18 85.09 0)
 			(effects
@@
 			)
 		)
-		(property "Footprint" "Wire Holes:Vout Holed"
+		(property "Footprint" "Connector_Wire:SolderWirePad_1x01_SMD_5x10mm"
 			(at 266.7 93.98 0)
 			(effects
